File: PIA-module.kicad_pcb (KiCad board)
At the start: 2 copper layers, 99.8 x 99.8 mm, 19 parts, among them J1 Conn_01x02_Male, J10 Conn_01x32, J11 Conn_01x32, J2 Conn_01x02_Male, J3 Conn_02x30_Odd_Even, J4 Conn_01x32, J5 Conn_01x32, J6 Conn_01x32, J7 Conn_01x32, J8 Conn_01x32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

Commit message: add mapped memory lane
Parts:
- removed the U3 at (148.9, 133.3)
- moved U2 15.4 mm to (148.9, 133.3)
- renumbered U4 to U3, U5 to U4
Connections:
- J3 pad 27: unconnected-(J3-Pad27) -> MAPPED_MEM
- U2 pad 1: A8 -> +5V
- U2 pad 10: A13 -> +5V
- U2 pad 12: A14 -> MAPPED_MEM
- U2 pad 13: A15 -> Net-(U2-Pad13)
- U2 pad 2: A9 -> Net-(U1-Pad4)
- U2 pad 4: A10 -> Net-(U1-Pad10)
- U2 pad 5: A11 -> Net-(U1-Pad13)
- U2 pad 6: Net-(U2-Pad6) -> Net-(U2-Pad13)
- U2 pad 9: A12 -> +5V
- U3 pad 2: Net-(U3-Pad8) -> Net-(U2-Pad8)
Routing:
- net ~{IRQ}: track 84.9 -> 0.00 mm
- net PB1: track 76.2 -> 0.00 mm
- net Q1: track 67.6 -> 0.00 mm
- net Q2: track 63.7 -> 0.00 mm
- net Q3: track 60.1 -> 0.00 mm
- net D5: track 58.7 -> 0.00 mm
- net E: track 54.9 -> 0.00 mm
- net Q4: track 54.8 -> 0.00 mm
- net Q5: track 51.9 -> 0.00 mm
- net Q6: track 49.9 -> 0.00 mm
- net PA7: track 49.8 -> 0.00 mm, vias 1 -> 0
- net Clock3: track 49.2 -> 0.00 mm
- net Q7: track 48.9 -> 0.00 mm
- net PA6: track 48.8 -> 0.00 mm, vias 1 -> 0
- net Q8: track 47.7 -> 0.00 mm
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
Commit message: add routing
Parts:
- removed the U3 at (141.5, 130.8)
- added JP1: FF00, Connector_PinHeader_2.54mm:PinHeader_1x03_P2.54mm_Vertical, F.Cu at (136.4, 130.9)
- added JP2: FF04, Connector_PinHeader_2.54mm:PinHeader_1x03_P2.54mm_Vertical, F.Cu at (132.7, 136.0)
- moved PL1 7.62 mm to (182.1, 94.2)
- moved PL2 7.54 mm to (138.6, 94.3)
- moved C1 3.64 mm to (129.6, 107.8)
- moved J8 2.90 mm to (102.4, 81.8)
- moved U5 2.86 mm to (181.6, 107.8)
- moved J5 2.85 mm to (102.4, 79.2)
- moved J10 2.80 mm to (102.4, 76.7)
- moved J7 2.75 mm to (102.4, 74.2)
- moved J4 2.70 mm to (102.4, 71.6)
- moved J11 2.65 mm to (102.4, 69.1)
- moved J9 2.60 mm to (102.4, 66.5)
- moved J6 2.55 mm to (102.4, 64.0)
- renumbered U2 to U3, U4 to U5
Connections:
- U1 pad 1: unconnected-(U1-Pad1) -> ~{CS2}
- U1 pad 2: unconnected-(U1-Pad2) -> Net-(U1-Pad2)
- U1 pad 3: unconnected-(U1-Pad3) -> Net-(U1-Pad2)
- U1 pad 5: A2 -> Net-(JP1-C)
- U3 pad 1: +5V -> Net-(JP2-C)
- U3 pad 8: Net-(U2-Pad8) -> Net-(U1-Pad2)
Routing:
- net Q2: track 0.00 -> 146.3 mm, vias 0 -> 3
- net Q4: track 0.00 -> 140.7 mm, vias 0 -> 3
- net Q1: track 0.00 -> 136.3 mm, vias 0 -> 3
- net Q6: track 0.00 -> 135.8 mm, vias 0 -> 3
- net Q3: track 0.00 -> 133.9 mm, vias 0 -> 3
- net Q8: track 0.00 -> 132.3 mm, vias 0 -> 3
- net Q7: track 0.00 -> 129.3 mm, vias 0 -> 3
- net Q5: track 0.00 -> 129.1 mm, vias 0 -> 3
- net ~{IRQ}: track 0.00 -> 83.5 mm, vias 0 -> 2
- net ~{RESET}: track 0.00 -> 66.6 mm, vias 0 -> 2
- net Clock3: track 0.00 -> 63.9 mm, vias 0 -> 1
- net E: track 0.00 -> 55.8 mm, vias 0 -> 1
- net PB7: track 0.00 -> 53.2 mm, vias 0 -> 1
- net PB6: track 0.00 -> 52.8 mm, vias 0 -> 1
- net CB1: track 0.00 -> 52.7 mm, vias 0 -> 2
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Other:
- board text added: "$FF00 JP1=1 JP2=2"
- board text added: "$FF04 JP1=2 JP2=1"
- board text added: "-3MHz"
- board text added: "1"
- board text added: "2"
- board text added: "Rev 1.1"
- board text added: "or $FF04-$FF07"
- board text removed: "-3MHz Clock"
