File: PIA-module.kicad_sch (KiCad schematic)
At the start: 6 parts, among them U1 74HC02, U2 74HC21, U3 74HC21, U4 74AHC1G04, U5 W65C21N

Commit message: add mapped memory lane
Parts:
- removed U2: 74HC21, Package_SO:SO-14_3.9x8.65mm_P1.27mm, symbol 74xx:74LS21
Connections:
- net +5V: now also U3.10
- net MAPPED_MEM: now reaches U3.12
Other:
- moved on the sheet: U1A

Commit message: add routing
Parts:
- removed U4: 74AHC1G04, Package_TO_SOT_SMD:SOT-353_SC-70-5, symbol 74xGxx:74AHC1G04
- added JP1: FF00, Connector_PinHeader_2.54mm:PinHeader_1x03_P2.54mm_Vertical, symbol Jumper:Jumper_3_Open
- added JP2: FF04, Connector_PinHeader_2.54mm:PinHeader_1x03_P2.54mm_Vertical, symbol Jumper:Jumper_3_Open
Connections:
- net +5V: now also JP2.3 (B); no longer U3.1
- net A2: now also JP1.3 (B), JP2.1 (A); no longer U1.5
- net GND: now also JP1.1 (A)
- net ~{CS2}: now also U1.1
- net at U3.8: now also U1.2, U1.3
- new net: JP2.2 (C), U3.1
- new net: JP1.2 (C), U1.5
- no-connect marks 3 -> 0
Other:
- moved on the sheet: U1A
